File: control_glove/pcb/control_glove_v0.1/control_glove_v0.1_dung_ki_hieu.kicad_sch (KiCad schematic)
At the start: 27 parts, among them J1 Conn_01x04_Female, J2 Conn_01x04_Female, J3 Conn_01x03_Female, J4 Conn_01x03_Female, J8 Conn_01x04_Female, P1 Power_Pins, SW3 SW_Push, SW5 SW_DIP_x01, U1 UART-RF433

Commit message: docs: Complete basic content of electric drawing
Parts:
- removed P1: Power_Pins, Connector_PinSocket_2.00mm:PinSocket_1x03_P2.00mm_Vertical, symbol hieu_lib:Power_Pins
- added BT1: Battery, symbol Device:Battery
- added J5, J6, J7: Conn_01x03_Male, symbol Connector:Conn_01x03_Male
- added J9: Conn_01x03_Female, Connector_PinSocket_2.00mm:PinSocket_1x03_P2.00mm_Vertical, symbol Connector:Conn_01x03_Female
- added Power1: Charging_module, symbol hieu_lib:Charging_module
- added RV1: R_Potentiometer, symbol Device:R_Potentiometer
- added SW1, SW2: SW_Push, hieu:resistor, symbol Switch:SW_Push
Connections:
- net GNDREF: now also J9.2 (Pin_2)
- net at SW5.1: now also J9.1 (Pin_1)
- net at SW_6.1: now also J9.3 (Pin_3)
- new net: J7.1 (Pin_1), Power1.3 (5V_OUT)
- new net: J7.2 (Pin_2), Power1.4 (GND)
- new net: J7.3 (Pin_3), Power1.5 (K)
- new net: J5.3 (Pin_3), SW1.1, SW2.1
- new net: J5.2 (Pin_2), SW1.2
- new net: J6.3 (Pin_3), RV1.1
- new net: J6.2 (Pin_2), RV1.2
- new net: J6.1 (Pin_1), RV1.3
- new net: BT1.1 (+), Power1.7 (V_BAT+)
- new net: BT1.2 (-), Power1.6 (V_BAT-)
- new net: J5.1 (Pin_1), SW2.2
- no-connect marks 23 -> 27
Other:
- note removed: "MAIN MODULE"
- note removed: "SHOULDER MODULE"
- moved on the sheet: D1, D2, IMU1, J1, J2, J3, J4, J8, JP1, MARG1, MCU1, R1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
